File: project-2.kicad_pcb (KiCad board)
At the start: 2 copper layers, 63.2 x 76.5 mm, 6 parts, among them M1 Motor_DC, SW1 SW_Push

Commit message: fix circuit 2
Parts:
- moved RV2 5.75 mm to (216.5, 82.0), turned to 180 degrees
- moved M1 3.81 mm to (209.5, 71.7), turned to 0 degrees
Connections:
- D1 pad 1: Net-(D1-K) -> Net-(BT1--)
- M1 pad 1: Net-(BT1--) -> Net-(M1-+)
- M1 pad 2: Net-(D1-K) -> Net-(BT1--)
- RV2 pad 1: Net-(BT1--) -> Net-(M1-+)
- RV2 pad 2: unconnected-(RV2-Pad2) -> Net-(RV1-Pad2)
Routing:
- net Net-(RV1-Pad2): track 11.9 -> 64.1 mm
- net Net-(BT1--): track 28.9 -> 45.2 mm
- net Net-(D1-K): track 16.1 -> 0.00 mm
- net Net-(M1-+): track 0.00 -> 13.2 mm
