File: project-2.kicad_pcb (KiCad board)
At the start: 2 copper layers, 63.2 x 76.5 mm, 6 parts, among them M1 Motor_DC, SW1 SW_Push

Commit message: cat
Other:
- board size 63.2 x 76.5 mm -> 63.5 x 80.1 mm
