File: project-2.kicad_sch (KiCad schematic)
At the start: 6 parts, among them M1 Motor_DC, SW1 SW_Push

Commit message: fix circuit 2
Connections:
- net at RV1.2, SW1.2: now also RV2.2
- net at M1.1 (+), RV2.1: no longer BT1.2 (-)
- net at D1.1 (K), M1.2 (-): now also BT1.2 (-)
Other:
- moved on the sheet: D1, M1
Changed lines of the file:
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@@
 	(paper "A4")
 	(junction
-		(at 110.49 45.72)
+		(at 129.54 53.34)
 		(diameter 0)
 		(color 0 0 0 0)
 	)
+	(junction
+		(at 62.23 60.96)
+		(diameter 0)
+		(color 0 0 0 0)
+	)
 	(wire
 		(pts
@@
 	(wire
 		(pts
-			(xy 101.6 45.72) (xy 110.49 45.72)
-		)
-		(stroke
-			(width 0)
-			(type default)
-		)
-	)
-	(wire
-		(pts
 			(xy 78.74 53.34) (xy 101.6 53.34)
 		)
@@
 	(wire
 		(pts
-			(xy 101.6 53.34) (xy 101.6 45.72)
+			(xy 129.54 66.04) (xy 129.54 53.34)
+		)
+		(stroke
+			(width 0)
+			(type default)
+		)
+	)
+	(wire
+		(pts
+			(xy 129.54 53.34) (xy 129.54 44.45)
 		)
 		(stroke
@@
 	(wire
 		(pts
-			(xy 110.49 44.45) (xy 110.49 45.72)
-		)
-		(stroke
-			(width 0)
-			(type default)
-		)
-	)
-	(wire
-		(pts
-			(xy 36.83 44.45) (xy 110.49 44.45)
-		)
-		(stroke
-			(width 0)
-			(type default)
-		)
-	)
-	(wire
-		(pts
-			(xy 59.69 49.53) (xy 74.93 49.53)
-		)
-		(stroke
-			(width 0)
-			(type default)
-		)
-	)
-	(wire
-		(pts
-			(xy 78.74 66.04) (xy 104.14 66.04)
+			(xy 62.23 49.53) (xy 74.93 49.53)
+		)
+		(stroke
+			(width 0)
+			(type default)
+		)
+	)
+	(wire
+		(pts
+			(xy 36.83 44.45) (xy 129.54 44.45)
+		)
+		(stroke
+			(width 0)
+			(type default)
+		)
+	)
+	(wire
+		(pts
+			(xy 78.74 66.04) (xy 101.6 66.04)
 		)
 		(stroke
@@
 	(wire
 		(pts
-			(xy 111.76 58.42) (xy 110.49 58.42)
-		)
-		(stroke
-			(width 0)
-			(type default)
-		)
-	)
-	(wire
-		(pts
-			(xy 59.69 60.96) (xy 59.69 49.53)
-		)
-		(stroke
-			(width 0)
-			(type default)
-		)
-	)
-	(wire
-		(pts
-			(xy 111.76 66.04) (xy 111.76 58.42)
+			(xy 109.22 66.04) (xy 129.54 66.04)
+		)
+		(stroke
+			(width 0)
+			(type default)
+		)
+	)
+	(wire
+		(pts
+			(xy 114.3 53.34) (xy 129.54 53.34)
+		)
+		(stroke
+			(width 0)
+			(type default)
+		)
+	)
+	(wire
+		(pts
+			(xy 62.23 60.96) (xy 62.23 49.53)
 		)
 		(stroke
@@
 	(symbol
 		(lib_id "Device:LED")
-		(at 107.95 66.04 180)
+		(at 105.41 66.04 180)
 		(unit 1)
 		(exclude_from_sim no)
@@
 		(fields_autoplaced yes)
 		(property "Reference" "D1"
-			(at 109.5375 58.42 0)
+			(at 106.9975 58.42 0)
 			(effects
 				(font
@@
 		)
 		(property "Value" "LED"
-			(at 109.5375 60.96 0)
+			(at 106.9975 60.96 0)
 			(effects
 				(font
@@
 		)
 		(property "Footprint" "LED_THT:LED_D5.0mm"
-			(at 107.95 66.04 0)
+			(at 105.41 66.04 0)
 			(effects
 				(font
@@
 		)
 		(property "Datasheet" "~"
-			(at 107.95 66.04 0)
+			(at 105.41 66.04 0)
 			(effects
 				(font
@@
 		)
 		(property "Description" "Light emitting diode"
-			(at 107.95 66.04 0)
+			(at 105.41 66.04 0)
 			(effects
 				(font
@@
 		)
 		(property "Sim.Pins" "1=K 2=A"
-			(at 107.95 66.04 0)
+			(at 105.41 66.04 0)
 			(effects
 				(font
@@
 	(symbol
 		(lib_id "Motor:Motor_DC")
-		(at 110.49 50.8 0)
+		(at 106.68 53.34 90)
 		(unit 1)
 		(exclude_from_sim no)
@@
 		(fields_autoplaced yes)
 		(property "Reference" "M1"
-			(at 115.57 52.0699 0)
-			(effects
-				(font
-					(size 1.27 1.27)
-				)
-				(justify left)
+			(at 109.22 45.72 90)
+			(effects
+				(font
+					(size 1.27 1.27)
+				)
 			)
 		)
 		(property "Value" "Motor_DC"
-			(at 115.57 54.6099 0)
-			(effects
-				(font
-					(size 1.27 1.27)
-				)
-				(justify left)
+			(at 109.22 48.26 90)
+			(effects
+				(font
+					(size 1.27 1.27)
+				)
 			)
 		)
 		(property "Footprint" "Connector_PinHeader_2.54mm:PinHeader_1x02_P2.54mm_Vertical"
-			(at 110.49 53.086 0)
+			(at 108.966 53.34 0)
 			(effects
 				(font
@@
 		)
 		(property "Datasheet" "~"
-			(at 110.49 53.086 0)
+			(at 108.966 53.34 0)
 			(effects
 				(font
@@
 		)
 		(property "Description" "DC Motor"
-			(at 110.49 50.8 0)
-			(effects
-				(font
+			(at 106.68 53.34 0)
+			(effects
+				(font
